Commit message: feat: add kitchen task

File: urdf/lekiwi/lekiwi.urdf (robot description, URDF)
Before this commit: robot LeKiwi, 45 links, 44 joints
Links:
- link base_plate_layer1_v5: mass 1.9468624348344596 -> 10.0

Commit message: fix: small physical logic fixed

File: urdf/lekiwi/lekiwi.urdf (robot description, URDF)
Before this commit: robot LeKiwi, 45 links, 44 joints
Links:
- link base_plate_layer1_v5: mass 10.0 -> 150.0
